Commit message: update

File: datasave/urdf/ur5e_extract_calibrated.urdf (robot description, URDF)
Before this commit: robot ur5e, 12 links, 11 joints
Links:
- link base_link_inertia: geometry collision mesh filename=/home/yuth/robotics_dev/tosave/ur5e/collision/base.stl; visual mesh filename=/home/yuth/robotics_dev/tosave/ur5e/visual/base.dae
- link forearm_link: geometry collision mesh filename=/home/yuth/robotics_dev/tosave/ur5e/collision/forearm.stl; visual mesh filename=/home/yuth/robotics_dev/tosave/ur5e/visual/forearm.dae
- link shoulder_link: geometry collision mesh filename=/home/yuth/robotics_dev/tosave/ur5e/collision/shoulder.stl; visual mesh filename=/home/yuth/robotics_dev/tosave/ur5e/visual/shoulder.dae
- link upper_arm_link: geometry collision mesh filename=/home/yuth/robotics_dev/tosave/ur5e/collision/upperarm.stl; visual mesh filename=/home/yuth/robotics_dev/tosave/ur5e/visual/upperarm.dae
- link wrist_1_link: geometry collision mesh filename=/home/yuth/robotics_dev/tosave/ur5e/collision/wrist1.stl; visual mesh filename=/home/yuth/robotics_dev/tosave/ur5e/visual/wrist1.dae
- link wrist_2_link: geometry collision mesh filename=/home/yuth/robotics_dev/tosave/ur5e/collision/wrist2.stl; visual mesh filename=/home/yuth/robotics_dev/tosave/ur5e/visual/wrist2.dae
- link wrist_3_link: geometry collision mesh filename=/home/yuth/robotics_dev/tosave/ur5e/collision/wrist3.stl; visual mesh filename=/home/yuth/robotics_dev/tosave/ur5e/visual/wrist3.dae
